File: hw/usb-pd/MAX25240A.kicad_sch (KiCad schematic)
At the start: 24 parts

Commit message: Preliminary PCB layout, calculated compensation filter and feedback network for MAX25240
Parts:
- added D4: V8PL6-M3/86A, footprints:TMBS-TO-277A, symbol Device:D_Schottky_Small
- C10: renamed from C?; value Cc -> 4.7nF 16V
- C12: renamed from C?; value Cf -> 310pF 16V
- L1: renamed from L?; value L_Small -> 10uH 8.4A; footprint Inductor_SMD:L_2512_6332Metric_Pad1.52x3.35mm_HandSolder -> footprints:BPSC00131380100M00
- R10: renamed from R?; value Rfbb3 -> 3k
- R11: renamed from R?; value Rfbb4 -> 5k1
- R12: renamed from R?; value Rfbb5 -> 18k
- R13: renamed from R?; value Rfbt -> 200k
- R7: renamed from R?; value Rc -> 47k
- R8: renamed from R?; value Rfbb1 -> 8k2
- R9: renamed from R?; value Rfbb2 -> 3k
- gave numbers to parts that had none: 14
Connections:
- net Vout: now also D4.1 (K)
- net at C9.1, L1.2, U2.8 (LX2): now also D4.2 (A)
- net at C11.1, U2.21 (VCC): now also U2.18 (SPS); no longer U2.19 (SYNC)
